File: fancontroller/fancontroller.kicad_pcb (KiCad board)
At the start: 2 copper layers, 60 x 60 mm, 24 parts, among them J1 Power, J2 Serial Conn, M1 FAN0, M2 FAN0, M3 FAN0, M4 FAN0, M5 FAN0, M6 FAN0, SW1 SW_Push, U2 ESP32-WROOM-32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

Commit message: First pcb iteration done
Connections:
- U2 pad 39: unconnected-(U2-GND-Pad39)_2 -> GND
- U2 pad 5: TMP1 -> TMP2
- U2 pad 6: TMP2 -> TMP1
Routing:
- net +3.3V: track 153.3 -> 24.8 mm, vias 0 -> 4
- net Tacho3: track 0.00 -> 49.0 mm, vias 0 -> 2
- net Tacho4: track 0.00 -> 48.3 mm, vias 0 -> 3
- net PWM3: track 0.00 -> 44.4 mm, vias 0 -> 2
- net TMP3: track 11.0 -> 49.1 mm, vias 0 -> 1
- net TMP2: track 7.71 -> 44.9 mm, vias 0 -> 1
- net TMP0: track 6.11 -> 40.1 mm, vias 0 -> 1
- net TMP1: track 8.85 -> 41.9 mm, vias 0 -> 1
- net PWM4: track 16.2 -> 45.1 mm, vias 0 -> 3
- net PWM2: track 47.1 -> 43.2 mm
- net (no net): vias 1 -> 0

Commit message: Update pcb
Parts:
- added REF**: Symbol_GNU-Logo_SilkscreenTop, Symbol:Symbol_GNU-Logo_SilkscreenTop, F.Cu at (123.5, 97.0)
