File: fancontroller/fancontroller.kicad_sch (KiCad schematic)
At the start: 43 parts, among them J1 Power, J2 Serial Conn, M1 FAN0, M2 FAN0, M3 FAN0, M4 FAN0, M5 FAN0, M6 FAN0, Q1 AO3400A, Q10 AO3401A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

Commit message: Move motor connection out in hirarchical sheet
Parts:
- removed M1, M2, M3, M4, M5, M6: FAN0, Connector:FanPinHeader_1x04_P2.54mm_Vertical, symbol Motor:Fan_Tacho_PWM
- removed Q1, Q11, Q3, Q5, Q7, Q9: AO3400A, Package_TO_SOT_SMD:SOT-23, symbol Transistor_FET:AO3400A
- removed Q10, Q12, Q2, Q4, Q6, Q8: AO3401A, Package_TO_SOT_SMD:SOT-23, symbol Transistor_FET:AO3401A
- removed R10, R11, R6, R7, R8, R9: 10k, Resistor_SMD:R_0805_2012Metric, symbol Device:R
- added U3: ESP32, DJCustom:QFN-48-1EP_6x6mm_P0.4mm_EP4.3x4.3mm, symbol PCM_Espressif:ESP32
- renumbered C6 to C1, C8 to C2, C9 to C3, U3 to U1
Connections:
- new net: U3.1 (VDDA), U3.43 (VDDA), U3.46 (VDDA)
- new net: U3.3 (VDD3P3), U3.4 (VDD3P3)
Other:
- added sheet Motor_Connections (motor_conn.kicad_sch)
- title: (none) -> ESP Fancontroller
